File: -009_012/Xbox-PMS.kicad_sch (KiCad schematic)
At the start: 112 parts, among them IC1 SIC437BED-T1-GE3, IC3 SIC437BED-T1-GE3, IC4 SIC437BED-T1-GE3, J2 USB_C_Receptacle_USB2.0_16P, J3 Jack-DC, J6 Conn_01x04_Pin, J7 Conn_01x04_Pin, U1 TVS2200DRV, U2 TPS25750, U3 CAT24C512

Commit message: + Update design to Universal, 1 PCB covers all 3 Xbox Motherboard Revisions now. + Clean up schematic refdes + Clean up zone outlines + Add 009/012 schematic
Parts:
- added C1, C3, C5: 22uF, Capacitor_SMD:C_1210_3225Metric, symbol Device:C_Small
- added C12: 1uF, Capacitor_SMD:C_0402_1005Metric, symbol Device:C_Small
- added C15: 4.7uF, Capacitor_SMD:C_0603_1608Metric, symbol Device:C_Small
- added C19: 0.1uF, Capacitor_SMD:C_0402_1005Metric, symbol Device:C_Small
- added C21, C24, C27: 47uF, Capacitor_SMD:C_1210_3225Metric, symbol Device:C_Small
- added C30, C33, C36, C39, C7: 22uF, Capacitor_SMD:C_0603_1608Metric, symbol Device:C_Small
- added C42: 0.1uF, Capacitor_SMD:C_0603_1608Metric, symbol Device:C_Small
- added IC2: SIC437BED-T1-GE3, Xbox-PMS:SIC437BEDT1GE3, symbol SIC437BED-T1-GE3:SIC437BED-T1-GE3
- added J8, J9: Conn_01x01_Pin, TestPoint:TestPoint_Pad_1.5x1.5mm, symbol Connector:Conn_01x01_Pin
- added L1: 780nH, Inductor_SMD:L_7.3x7.3_H4.5, symbol Device:L_Small
- added R1, R12: 10K, Resistor_SMD:R_0402_1005Metric, symbol Device:R_Small
- added R13: 2.2R, Resistor_SMD:R_0402_1005Metric, symbol Device:R_Small
- added R14: 45K, Resistor_SMD:R_0402_1005Metric, symbol Device:R_Small
- added R3: 100K, Resistor_SMD:R_0402_1005Metric, symbol Device:R_Small
- added R4: 499K, Resistor_SMD:R_0402_1005Metric, symbol Device:R_Small
- added TP3, TP4: TestPoint, Xbox-PMS:pad, symbol Connector:TestPoint
- R17: value 18.7K -> 45K; MPN CRCW040218K7FKEDC -> P-0402H4502BGTS
Connections:
- net EN: now also IC2.19 (EN), J9.1 (Pin_1)
- net GND: now also C1.2, C12.1, C15.1, C21.1, C24.2, C27.2, C3.2, C30.2, C33.2, C36.2, C39.2, C42.2, C5.2, C7.2, IC2.13 (PGND), IC2.16 (AGND), IC2.25 (AGND), IC2.27 (PGND), IC2.29 (PGND), IC2.3 (PGND), IC2.4 (PGND), R12.2, TP4.1
- net PGOOD: now also IC2.14 (P_GOOD), J8.1 (Pin_1), R1.1
- net VBUS-SAFE: now also C1.1, C3.1, C5.1, C7.1, IC2.1 (VIN), IC2.2 (VIN), IC2.22 (VIN), IC2.26 (VIN)
- net VDD: now also C12.2, C15.2, IC2.12 (V_DRV), IC2.15 (VDD), R1.2, R3.2, R4.1
- new net: IC2.17 (FB), R12.1, R14.2
- new net: IC2.20 (MODE2), R4.2
- new net: IC2.21 (MODE1), R3.1
- new net: C19.1, IC2.23 (BOOT)
- new net: IC2.24 (PHASE), R13.1
- new net: IC2.30 (SW), IC2.5 (SW), IC2.6 (SW), IC2.7 (SW), IC2.8 (SW), IC2.9 (SW), L1.1
- new net: C19.2, R13.2
- new net 3V3SW: C21.2, C24.1, C27.1, C30.1, C33.1, C36.1, C39.1, C42.1, IC2.18 (VOUT), L1.2, R14.1, TP3.1
Other:
- note added: "3V3"
- note added: "3V3SB"
- note removed: "5VSB"
- moved on the sheet: C64, C65, C66, C67, C68, C69, C70, C71, C72, C73, C74, C75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

Commit message: Fix value of R15 in -009_012 schematic
Parts:
- R15: value 2.55K -> 10K
Changed lines of the file:
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@@
 			)
 		)
-		(property "Value" "2.55K"
+		(property "Value" "10K"
 			(at 116.84 225.425 0)
 			(effects
